File: zigbee-led-controller.kicad_sch (KiCad schematic)
At the start: 61 parts, among them J1 SWD Header, J2 UART, J3 12V_Input, J4 LED_Connector, J5 5V_Input, J6 USB_B_Micro, J7 2.1x5.5mm, Q1 IRLML0040TRPbF, Q2 IRLML0040TRPbF, Q3 IRLML0040TRPbF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

Commit message: Added GRAVITECH_CON-SOCJ-2155 footprint for the barrel connector.
Parts:
- J7: footprint (none) -> Library:GRAVITECH_CON-SOCJ-2155; MFP (none) -> CON-SOCJ-2155; SUPPLIER (none) -> Mouser; SUPPLIER_PN (none) -> 992-CON-SOCJ-2155
Changed lines of the file:
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@@
       (effects (font (size 1.27 1.27)))
     )
-    (property "Footprint" "" (at 39.37 77.851 0)
+    (property "Footprint" "Library:GRAVITECH_CON-SOCJ-2155" (at 39.37 77.851 0)
       (effects (font (size 1.27 1.27)) hide)
     )
-    (property "Datasheet" "~" (at 39.37 77.851 0)
+    (property "Datasheet" "https://www.gravitech.us/poja2x51.html" (at 39.37 77.851 0)
       (effects (font (size 1.27 1.27)) hide)
     )
+    (property "MFN" "" (at 38.1 76.835 0)
+      (effects (font (size 1.27 1.27)) hide)
+    )
+    (property "MFP" "CON-SOCJ-2155" (at 38.1 76.835 0)
+      (effects (font (size 1.27 1.27)) hide)
+    )
+    (property "SUPPLIER" "Mouser" (at 38.1 76.835 0)
+      (effects (font (size 1.27 1.27)) hide)
+    )
+    (property "SUPPLIER_PN" "992-CON-SOCJ-2155" (at 38.1 76.835 0)
+      (effects (font (size 1.27 1.27)) hide)
+    )
+    (property "ALT_SUPPLIER" "" (at 38.1 76.835 0)
+      (effects (font (size 1.27 1.27)) hide)
+    )
+    (property "ALT_SUPPLIER_PN" "" (at 38.1 76.835 0)
+      (effects (font (size 1.27 1.27)) hide)
+    )
+    (property "SUPPLIER_LINK" "" (at 38.1 76.835 0)
+      (effects (font (size 1.27 1.27)) hide)
+    )
+    (property "ALT_SUPPLIER_LINK" "" (at 38.1 76.835 0)
+      (effects (font (size 1.27 1.27)) hide)
+    )

Commit message: PCB Initial placement
Parts:
- J1, J2: footprint Connector_PinHeader_2.54mm:PinHeader_1x02_P2.54mm_Horizontal -> Connector_PinHeader_2.54mm:PinHeader_1x02_P2.54mm_Vertical
- J3: footprint Connector_Molex:Molex_KK-396_A-41792-0004_1x04_P3.96mm_Horizontal -> Connector_PinHeader_2.54mm:PinHeader_1x04_P2.54mm_Horizontal
- J4: footprint Connector_PinHeader_2.54mm:PinHeader_1x03_P2.54mm_Vertical -> Connector_PinHeader_2.54mm:PinHeader_1x05_P2.54mm_Vertical
- J5: footprint Connector_Molex:Molex_KK-396_A-41792-0002_1x02_P3.96mm_Horizontal -> Connector_PinHeader_2.54mm:PinHeader_1x02_P2.54mm_Horizontal
Changed lines of the file:
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@@
       (effects (font (size 1.27 1.27)))
     )
-    (property "Footprint" "Connector_Molex:Molex_KK-396_A-41792-0004_1x04_P3.96mm_Horizontal" (at 34.925 92.075 0)
+    (property "Footprint" "Connector_PinHeader_2.54mm:PinHeader_1x04_P2.54mm_Horizontal" (at 34.925 92.075 0)
       (effects (font (size 1.27 1.27)) hide)
     )
@@
       (effects (font (size 1.27 1.27)) (justify right))
     )
-    (property "Footprint" "Connector_PinHeader_2.54mm:PinHeader_1x02_P2.54mm_Horizontal" (at 212.09 22.86 0)
+    (property "Footprint" "Connector_PinHeader_2.54mm:PinHeader_1x02_P2.54mm_Vertical" (at 212.09 22.86 0)
       (effects (font (size 1.27 1.27)) hide)
     )
@@
       (effects (font (size 1.27 1.27)) (justify left))
     )
-    (property "Footprint" "Connector_PinHeader_2.54mm:PinHeader_1x02_P2.54mm_Horizontal" (at 276.225 73.66 0)
+    (property "Footprint" "Connector_PinHeader_2.54mm:PinHeader_1x02_P2.54mm_Vertical" (at 276.225 73.66 0)
       (effects (font (size 1.27 1.27)) hide)
     )
@@
       (effects (font (size 1.27 1.27)))
     )
-    (property "Footprint" "Connector_Molex:Molex_KK-396_A-41792-0002_1x02_P3.96mm_Horizontal" (at 34.925 118.11 0)
+    (property "Footprint" "Connector_PinHeader_2.54mm:PinHeader_1x02_P2.54mm_Horizontal" (at 34.925 118.11 0)
       (effects (font (size 1.27 1.27)) hide)
     )
     (property "Datasheet" "~" (at 34.925 118.11 0)
+      (effects (font (size 1.27 1.27)) hide)
+    )
+    (property "MFN" "" (at 34.925 118.11 0)
+      (effects (font (size 1.27 1.27)) hide)
+    )
+    (property "MFP" "" (at 34.925 118.11 0)
+      (effects (font (size 1.27 1.27)) hide)
+    )
+    (property "SUPPLIER" "" (at 34.925 118.11 0)
+      (effects (font (size 1.27 1.27)) hide)
+    )
+    (property "SUPPLIER_PN" "" (at 34.925 118.11 0)
+      (effects (font (size 1.27 1.27)) hide)
+    )
+    (property "ALT_SUPPLIER" "" (at 34.925 118.11 0)
+      (effects (font (size 1.27 1.27)) hide)
+    )
+    (property "ALT_SUPPLIER_PN" "" (at 34.925 118.11 0)
+      (effects (font (size 1.27 1.27)) hide)
+    )
+    (property "SUPPLIER_LINK" "" (at 34.925 118.11 0)
+      (effects (font (size 1.27 1.27)) hide)
+    )
+    (property "ALT_SUPPLIER_LINK" "" (at 34.925 118.11 0)
       (effects (font (size 1.27 1.27)) hide)
     )
@@
       (effects (font (size 1.27 1.27)) (justify left))
     )
-    (property "Footprint" "Connector_PinHeader_2.54mm:PinHeader_1x03_P2.54mm_Vertical" (at 266.7 114.3 0)
-      (effects (font (size 1.27 1.27)) hide)
-    )
+    (property "Footprint" "Connector_PinHeader_2.54mm:PinHeader_1x05_P2.54mm_Vertical" (at 266.7 114.3 0)
+      (effects (font (size 1.27 1.27)) hide)
+    )

Commit message: Routing done, first pass anyway.
Connections:
- net B_LED_d: now also U2.3 (A10/0.28); no longer U2.4 (A11/0.29)
- net G_LED_d: now also U2.4 (A11/0.29); no longer U2.2 (A4/0.03_H)
- net R_LED_d: now also U2.9 (A7_SCK/1.13); no longer U2.1 (A2/0.02_H)
- net WP: now also U2.1 (A2/0.02_H); no longer U2.3 (A10/0.28)
- net W_LED_d: now also U2.2 (A4/0.03_H); no longer U2.9 (A7_SCK/1.13)
Changed lines of the file:
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@@
     (stroke (width 0) (type default))
   )
-  (wire (pts (xy 185.42 48.26) (xy 194.31 48.26))
+  (wire (pts (xy 156.845 48.26) (xy 194.31 48.26))
     (stroke (width 0) (type default))
   )
@@
     (stroke (width 0) (type default))
   )
-  (wire (pts (xy 156.845 53.34) (xy 156.845 46.355))
-    (stroke (width 0) (type default))
-  )
   (wire (pts (xy 276.86 55.88) (xy 276.86 57.785))
     (stroke (width 0) (type default))
   )
+  (wire (pts (xy 156.845 48.26) (xy 156.845 46.355))
+    (stroke (width 0) (type default))
+  )
   (wire (pts (xy 88.265 89.535) (xy 90.805 89.535))
     (stroke (width 0) (type default))
@@
     (stroke (width 0) (type default))
   )
+  (wire (pts (xy 185.42 53.34) (xy 194.31 53.34))
+    (stroke (width 0) (type default))
+  )
   (wire (pts (xy 202.565 148.59) (xy 202.565 156.845))
     (stroke (width 0) (type default))
@@
   )
   (wire (pts (xy 210.82 116.84) (xy 210.82 119.38))
-    (stroke (width 0) (type default))
-  )
-  (wire (pts (xy 156.845 53.34) (xy 194.31 53.34))
     (stroke (width 0) (type default))
   )
@@
     (effects (font (size 1.27 1.27)) (justify left bottom))
   )
-  (label "G_LED_d" (at 185.42 50.8 180) (fields_autoplaced)
+  (label "G_LED_d" (at 185.42 55.88 180) (fields_autoplaced)
     (effects (font (size 1.27 1.27)) (justify right bottom))
   )
@@
     (effects (font (size 1.27 1.27)) (justify left bottom))
   )
-  (label "B_LED_d" (at 185.42 55.88 180) (fields_autoplaced)
+  (label "B_LED_d" (at 185.42 53.34 180) (fields_autoplaced)
     (effects (font (size 1.27 1.27)) (justify right bottom))
   )
-  (label "R_LED_d" (at 185.42 48.26 180) (fields_autoplaced)
+  (label "R_LED_d" (at 244.475 60.96 0) (fields_autoplaced)
+    (effects (font (size 1.27 1.27)) (justify left bottom))
+  )
+  (label "SWDIO" (at 212.09 39.37 90) (fields_autoplaced)
+    (effects (font (size 1.27 1.27)) (justify left bottom))
+  )
+  (label "B_LED_d" (at 135.89 132.715 0) (fields_autoplaced)
+    (effects (font (size 1.27 1.27)) (justify left bottom))
+  )
+  (label "G_LED_d" (at 135.89 126.365 0) (fields_autoplaced)
+    (effects (font (size 1.27 1.27)) (justify left bottom))
+  )
+  (label "RESETn" (at 218.44 26.035 0) (fields_autoplaced)
+    (effects (font (size 1.27 1.27)) (justify left bottom))
+  )
+  (label "W_LED_d" (at 185.42 50.8 180) (fields_autoplaced)
     (effects (font (size 1.27 1.27)) (justify right bottom))
   )
-  (label "SWDIO" (at 212.09 39.37 90) (fields_autoplaced)
-    (effects (font (size 1.27 1.27)) (justify left bottom))
-  )
-  (label "B_LED_d" (at 135.89 132.715 0) (fields_autoplaced)
-    (effects (font (size 1.27 1.27)) (justify left bottom))
-  )
-  (label "G_LED_d" (at 135.89 126.365 0) (fields_autoplaced)
-    (effects (font (size 1.27 1.27)) (justify left bottom))
-  )
-  (label "RESETn" (at 218.44 26.035 0) (fields_autoplaced)
-    (effects (font (size 1.27 1.27)) (justify left bottom))
-  )
-  (label "W_LED_d" (at 244.475 60.96 0) (fields_autoplaced)
-    (effects (font (size 1.27 1.27)) (justify left bottom))
-  )
   (label "LED_1" (at 245.11 55.88 0) (fields_autoplaced)
     (effects (font (size 1.27 1.27)) (justify left bottom))
   )
-  (label "WP" (at 177.8 53.34 0) (fields_autoplaced)
-    (effects (font (size 1.27 1.27)) (justify left bottom))
+  (label "WP" (at 185.42 48.26 180) (fields_autoplaced)
+    (effects (font (size 1.27 1.27)) (justify right bottom))
   )
   (label "TX" (at 268.605 76.2 0) (fields_autoplaced)

Commit message: Updated some footprints and finalized layout. Added better output connector and rst switch
Parts:
- C1, C2: SUPPLIER (none) -> Farnell; SUPPLIER_PN (none) -> 1740614
- C3, C4: SUPPLIER (none) -> Farnell; SUPPLIER_PN (none) -> 1907510
- C5: SUPPLIER (none) -> Farnell; SUPPLIER_PN (none) -> 2346927
- D1: SUPPLIER (none) -> Farnell; SUPPLIER_PN (none) -> 3796276
- D2, D3, D4: SUPPLIER (none) -> Farnell; SUPPLIER_PN (none) -> 3796316
- J3: DESCRIPTION (none) -> Pin Header, Right Angle, Wire-to-Board, 2.54 mm, 1 Rows, 4 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; MF (none) -> TE; MFP (none) -> 640457-4; SUPPLIER (none) -> Farnell; SUPPLIER_PN (none) -> 588738
- J4: DESCRIPTION (none) -> Wire-To-Board Terminal Block, 2.54 mm, 5 Ways, 30 AWG, 16 A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; MF (none) -> TE Connectivity; MFP (none) -> 282834-5; SUPPLIER (none) -> Farnell; SUPPLIER_PN (none) -> 2112483
- J5: DESCRIPTION (none) -> Pin Header, Wire-to-Board, 2.54 mm, 1 Rows, 2 Contacts, Thr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; SUPPLIER (none) -> Farnell; SUPPLIER_PN (none) -> 1675773
- J6: ALT_SUPPLIER (none) -> Wurth; ALT_SUPPLIER_PN (none) -> 710-629105150521; DESCRIPTION (none) -> USB Connectors WR-COM USB Micro SMT Type B Horiztl; SUPPLIER (none) -> Farnell; SUPPLIER_PN (none) -> 2470822
- L1: ALT_SUPPLIER (none) -> Mouser; ALT_SUPPLIER_PN (none) -> 70-IHLP1616ABR1R0M1A; DESCRIPTION (none) -> Power Inductors - SMD 1 ohms 20%; MF (none) -> Vishay; SUPPLIER (none) -> Farnell; SUPPLIER_PN (none) -> 2965604
- Q1, Q2, Q3, Q4: ALT_SUPPLIER (none) -> Mouser; ALT_SUPPLIER_PN (none) -> 942-IRLML0040TRPBF; SUPPLIER (none) -> Farnell; SUPPLIER_PN (none) -> 1831088
- R1, R2, R3: SUPPLIER (none) -> Farnell; SUPPLIER_PN (none) -> 2447385
- R10, R12, R6, R8: value 47 -> 47R; SUPPLIER (none) -> Farnell; SUPPLIER_PN (none) -> 2694082
- R11, R5, R7, R9: value 56 -> 56R; SUPPLIER (none) -> Farnell; SUPPLIER_PN (none) -> 2694086
- R13, R14, R15, R16: SUPPLIER (none) -> Farnell; SUPPLIER_PN (none) -> 2073349
- R17, R18, R19, R20: SUPPLIER (none) -> Farnell; SUPPLIER_PN (none) -> 2446547
- R21: SUPPLIER (none) -> Farnell; SUPPLIER_PN (none) -> 3392726
- R22: value 680 -> 680R; SUPPLIER (none) -> Farnell; SUPPLIER_PN (none) -> 2447419
- R23, R4: value 470 -> 470R; SUPPLIER (none) -> Farnell; SUPPLIER_PN (none) -> 2073508
- SW1: footprint Inductor_SMD:L_Vishay_IHLP-1616 -> SW_B3U-1000P; symbol Switch:SW_Push -> Project:B3U-1000P; ALT_SUPPLIER (none) -> mouser; ALT_SUPPLIER_PN (none) -> 653-B3U-1000P; AVAILABILITY (none) -> Unavailable; DESCRIPTION (none) -> Tactile Switch SPST-NO Top Actuated Surface Mount; MF (none) -> Omron; MFP (none) -> B3U-1000P; MP (none) -> B3U-1000P; PACKAGE (none) -> None; PRICE (none) -> None; SUPPLIER (none) -> Farnell; SUPPLIER_PN (none) -> 1333652
- TP1, TP2, TP3, TP4, TP5: ALT_SUPPLIER (none) -> Farnell; ALT_SUPPLIER_PN (none) -> 2301280; DESCRIPTION (none) -> Keystone THR testpoints; MF (none) -> Keystone; MFP (none) -> 5001; SUPPLIER (none) -> Mouser; SUPPLIER_PN (none) -> 534-5001
- U1: ALT_SUPPLIER (none) -> Mouser; ALT_SUPPLIER_PN (none) -> 556-AT24CS01-SSHM-T; SUPPLIER (none) -> Farnell; SUPPLIER_PN (none) -> 2920867
- U2: DESCRIPTION (none) -> Seeed XIAO BLE nRF52840; MF (none) -> Seeed; MFP (none) -> 104808; SUPPLIER (none) -> Pi Hut; SUPPLIER_LINK (none) -> https://thepihut.com/products/seeed-xiao-ble-nrf52840?varia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; SUPPLIER_PN (none) -> Seeed XIAO BLE nRF52840
- U3: ALT_SUPPLIER (none) -> Mouser; ALT_SUPPLIER_PN (none) -> 621-AP63205WU-7; SUPPLIER (none) -> Farnell; SUPPLIER_PN (none) -> 3518308
